Commit message: Add Elfin E05 freedrive and operator tooling

File: elfin_description/urdf/elfin5.urdf.xacro (robot description, xacro)
@@ -6,4 +6,12 @@
   <xacro:property name="PI" value="3.1415926535897931"/>
   <xacro:property name="density" value="3.09"/>
+  <!-- Defaults preserve the original model. The freedrive simulation passes
+       non-zero values to keep effort-controlled joints numerically damped. -->
+  <xacro:arg name="joint_damping_1" default="0.0" />
+  <xacro:arg name="joint_damping_2" default="0.0" />
+  <xacro:arg name="joint_damping_3" default="0.0" />
+  <xacro:arg name="joint_damping_4" default="0.0" />
+  <xacro:arg name="joint_damping_5" default="0.0" />
+  <xacro:arg name="joint_damping_6" default="0.0" />
   <link name="world"/>
   <joint name="world_base" type="fixed">
@@ -118,4 +126,5 @@
     <axis
       xyz="0 0 1" />
+    <dynamics damping="$(arg joint_damping_1)" friction="0.0" />
     <limit
       lower="-3.14"
@@ -176,4 +185,5 @@
     <axis
       xyz="0 0 1" />
+    <dynamics damping="$(arg joint_damping_2)" friction="0.0" />
     <limit
       lower="-2.35"
@@ -234,4 +244,5 @@
     <axis
       xyz="0 0 1" />
+    <dynamics damping="$(arg joint_damping_3)" friction="0.0" />
     <limit
       lower="-2.61"
@@ -292,4 +303,5 @@
     <axis
       xyz="0 0 1" />
+    <dynamics damping="$(arg joint_damping_4)" friction="0.0" />
     <limit
       lower="-3.14"
@@ -350,4 +362,5 @@
     <axis
       xyz="0 0 1" />
+    <dynamics damping="$(arg joint_damping_5)" friction="0.0" />
     <limit
       lower="-2.56"
@@ -408,4 +421,5 @@
     <axis
       xyz="0 0 1" />
+    <dynamics damping="$(arg joint_damping_6)" friction="0.0" />
     <limit
       lower="-3.14"

File: elfin_description/urdf/elfin_transmission.xacro (robot description, xacro)
@@ -1,8 +1,11 @@
 <?xml version="1.0"?>
 <robot xmlns:xacro="http://www.ros.org/wiki/xacro">
+    <!-- Gazebo freedrive tests override this to EffortJointInterface. -->
+    <xacro:arg name="transmission_hw_interface"
+               default="hardware_interface/PositionJointInterface" />
     <transmission name="elfin_joint1_trans">
       <type>transmission_interface/SimpleTransmission</type>
       <joint name="elfin_joint1">
-        <hardwareInterface>hardware_interface/PositionJointInterface</hardwareInterface>
+        <hardwareInterface>$(arg transmission_hw_interface)</hardwareInterface>
       </joint>
       <actuator name="elfin_joint1_motor">
@@ -13,5 +16,5 @@
       <type>transmission_interface/SimpleTransmission</type>
       <joint name="elfin_joint2">
-        <hardwareInterface>hardware_interface/PositionJointInterface</hardwareInterface>
+        <hardwareInterface>$(arg transmission_hw_interface)</hardwareInterface>
       </joint>
       <actuator name="elfin_joint2_motor">
@@ -22,5 +25,5 @@
       <type>transmission_interface/SimpleTransmission</type>
       <joint name="elfin_joint3">
-        <hardwareInterface>hardware_interface/PositionJointInterface</hardwareInterface>
+        <hardwareInterface>$(arg transmission_hw_interface)</hardwareInterface>
       </joint>
       <actuator name="elfin_joint3_motor">
@@ -31,5 +34,5 @@
       <type>transmission_interface/SimpleTransmission</type>
       <joint name="elfin_joint4">
-        <hardwareInterface>hardware_interface/PositionJointInterface</hardwareInterface>
+        <hardwareInterface>$(arg transmission_hw_interface)</hardwareInterface>
       </joint>
       <actuator name="elfin_joint4_motor">
@@ -40,5 +43,5 @@
       <type>transmission_interface/SimpleTransmission</type>
       <joint name="elfin_joint5">
-        <hardwareInterface>hardware_interface/PositionJointInterface</hardwareInterface>
+        <hardwareInterface>$(arg transmission_hw_interface)</hardwareInterface>
       </joint>
       <actuator name="elfin_joint5_motor">
@@ -49,5 +52,5 @@
       <type>transmission_interface/SimpleTransmission</type>
       <joint name="elfin_joint6">
-        <hardwareInterface>hardware_interface/PositionJointInterface</hardwareInterface>
+        <hardwareInterface>$(arg transmission_hw_interface)</hardwareInterface>
       </joint>
       <actuator name="elfin_joint6_motor">
